File: kicad/cdm324_v2/cdm324_v2.kicad_sch (KiCad schematic)
At the start: 37 parts, among them J2 Conn_01x03_Female, J4 Conn_02x04_Odd_Even, J5 Conn_02x04_Odd_Even, U1 LMP7731, U3 MAX9814, U4 NCP163ASN330T1G, U5 STM32F301K8Ux

Commit message: first stage changed, POR for segment controller
Parts:
- C4: value 200p -> 27p; Field4 https://www.digikey.com/product-detail/en/samsung-electro-m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 -> https://www.digikey.com/en/products/detail/yageo/CC0603JRNP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
- R3: value 130k -> 620k; Field4 https://www.digikey.com/product-detail/en/panasonic-electro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 -> (none)
Other:
- note added: "42.4dB"
- note added: "LPF 1.5Hz"
- note added: "measured low pass 7.7kHz (175km/h)"
- note removed: "42.3dB"
- note removed: "low pass 6.1kHz (138km/h)"
Changed lines of the file:
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@@
     (effects (font (size 1.27 1.27)) (justify left bottom))
   )
-  (text "low pass 6.1kHz\n    (138km/h)" (at 82.55 115.57 0)
+  (text "measured low pass 7.7kHz\n          (175km/h)" (at 78.74 115.57 0)
     (effects (font (size 1.27 1.27)) (justify left bottom))
   )
@@
     (effects (font (size 1.27 1.27)) (justify left bottom))
   )
-  (text "42.3dB" (at 92.71 99.06 0)
+  (text "LPF 1.5Hz" (at 68.58 88.9 0)
+    (effects (font (size 1.27 1.27)) (justify left bottom))
+  )
+  (text "42.4dB" (at 92.71 99.06 0)
     (effects (font (size 1.27 1.27)) (justify left bottom))
   )
@@
       (effects (font (size 1.27 1.27)))
     )
-    (property "Value" "200p" (at 95.25 107.95 90)
+    (property "Value" "27p" (at 95.25 107.95 90)
       (effects (font (size 1.27 1.27)))
     )
@@
       (effects (font (size 1.27 1.27)) hide)
     )
-    (property "Field4" "https://www.digikey.com/product-detail/en/samsung-electro-mechanics/CL10C201JB8NNNC/1276-2222-1-ND/3890308" (at 91.44 109.22 90)
+    (property "Field4" "https://www.digikey.com/en/products/detail/yageo/CC0603JRNPO9BN270/302797" (at 91.44 109.22 90)
       (effects (font (size 1.27 1.27)) hide)
     )
@@
       (effects (font (size 1.27 1.27)))
     )
-    (property "Value" "130k" (at 91.44 104.14 90)
+    (property "Value" "620k" (at 91.44 104.14 90)
       (effects (font (size 1.27 1.27)))
     )
@@
       (effects (font (size 1.27 1.27)) hide)
     )
-    (property "Field4" "https://www.digikey.com/product-detail/en/panasonic-electronic-components/ERJ-3EKF1303V/P130KHCT-ND/198154" (at 91.44 104.14 90)
-      (effects (font (size 1.27 1.27)) hide)
-    )
+    (property "Field4" "" (at 91.44 104.14 90)
+      (effects (font (size 1.27 1.27)) hide)
+    )

Commit message: correct resistor divider for jack output
Parts:
- R3: Field4 (none) -> https://www.digikey.com/en/products/detail/yageo/RC0603FR-0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
Changed lines of the file:
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@@
       (effects (font (size 1.27 1.27)) hide)
     )
-    (property "Field4" "" (at 91.44 104.14 90)
+    (property "Field4" "https://www.digikey.com/en/products/detail/yageo/RC0603FR-07620KL/727338" (at 91.44 104.14 90)
       (effects (font (size 1.27 1.27)) hide)
     )
